File: schematics/tower.sch (KiCad schematic (older format))
At the start: 14 parts, among them IC1 ESP32-SOLO-1, J1 Conn_01x02, J2 Conn_01x06, J3 Conn_01x09, J4 Conn_02x10_Odd_Even, SW1 SW_Push, SW2 SW_SPDT, U1 NCP1117-3.3_SOT223

Commit message: finished (I think) schematics for tower and controller
Parts:
- removed J1: Conn_01x02, Connector_PinHeader_1.00mm:PinHeader_1x02_P1.00mm_Vertical, symbol Connector_Generic:Conn_01x02
- removed J3: Conn_01x09, Connector_PinSocket_1.00mm:PinSocket_1x09_P1.00mm_Vertical, symbol Connector_Generic:Conn_01x09
- removed SW2: SW_SPDT, Button_Switch_THT:SW_Slide_1P2T_CK_OS102011MS2Q, symbol Switch:SW_SPDT
- removed U1: NCP1117-3.3_SOT223, Package_TO_SOT_SMD:SOT-223-3_TabPin2, symbol Regulator_Linear:NCP1117-3.3_SOT223
- added C3, C5: 100nF, Capacitor_SMD:C_0805_2012Metric, symbol Device:C
- added C4: 22uF, Capacitor_SMD:C_0805_2012Metric, symbol Device:C
- added D1: BAT760-7, Mouser:SOD2513X120N, symbol Mouser:BAT760-7
- added D2: LED, Mouser:APHCM2012QBCDF01, symbol Device:LED
- added J1: 216990-0003, Mouser:2169900003, symbol Mouser:216990-0003
- added J3: Conn_01x05, Connector_PinSocket_2.54mm:PinSocket_1x05_P2.54mm_Vertical, symbol Connector_Generic:Conn_01x05
- added J4: SD_Card, Connector_Card:SD_Kyocera_145638109211859+, symbol Connector:SD_Card
- added Q1, Q2: SS8050-G, Mouser:SOT95P240X115-3N, symbol Mouser:SS8050-G
- added R3, R4, R5: 10k, Resistor_SMD:R_0805_2012Metric, symbol Device:R
- added R6, R7: 0, Resistor_SMD:R_0201_0603Metric, symbol Device:R
- added SW2: SW_Push, Button_Switch_SMD:SW_SPST_CK_KXT3, symbol Switch:SW_Push
- C1, C2: value 100nF -> 0.1uF
- IC1: footprint RF_Module:ESP32-WROOM-32 -> Mouser:ESP32SOLO1; symbol controller-rescue:ESP32-SOLO-1-ESP-SOLO-1 -> tower-rescue:ESP32-SOLO-1-ESP-SOLO-1-controller-rescue
- R1: value 10k -> 20
- SW1: footprint Button_Switch_THT:SW_TH_Tactile_Omron_B3F-10xx -> Button_Switch_SMD:SW_SPST_CK_KXT3
- renumbered C3 to C6, C4 to C7, J4 to J5
Connections:
- net labels added: EN, PG, SDCLK, SDMISO, SDMOSI, SHDN, VIN, VOUT
- net labels removed: IO25, IO26, IO27
- wire segments 42 -> 78
Other:
- note added: "Boot PushButton"
- note added: "ESP32 module"
- note added: "IDC Box Header to display\n"
- note added: "MCU Power capacitor\n"
- note added: "Power LED"
- note added: "Program circuitry\n"
- note added: "Reset PushButton"
- note added: "Reset stabilizing"
- note added: "SD Card Reader\n"
- note added: "Switching Regulator"
- note added: "USB-C Power connector\n"
- note removed: "Boot pin"
- note removed: "Extra Connectors\n"
- note removed: "Linear regulator\n"
- note removed: "Reset pin\n"
- note removed: "Wall charger connections"
- moved on the sheet: J2
