File: schematics/car.kicad_sch (KiCad schematic)
At the start: 37 parts, among them IC1 ESP32-SOLO-1, J1 Conn_01x09_Female, J2 Conn_01x04_Male, J3 Conn_01x02_Female, J4 Conn_01x06_Female, J5 Conn_01x05_Female, J6 Conn_01x05_Female, Q1 SS8050-G, Q2 SS8050-G, SW1 SW_Push, SW2 SW_Push, U1 L298HN

Commit message: final pcbs and schematics
Parts:
- added C7: 100uF, Capacitor_THT:CP_Radial_D8.0mm_P5.00mm, symbol Device:C
- added H1, H2, H3, H4: MountingHole, MountingHole:MountingHole_2.5mm_Pad, symbol Mechanical:MountingHole
- added R11, R12: 10k, Resistor_SMD:R_0805_2012Metric, symbol Device:R
- C3: value 10uF -> 100uF; footprint Capacitor_THT:CP_Radial_D4.0mm_P1.50mm -> Capacitor_THT:CP_Radial_D8.0mm_P5.00mm
Connections:
- net 3.3V: now also R11.2, R12.2; no longer J4.4 (Pin_4)
- net EN: now also R12.1
- net GND: now also C7.1
- net GPIO0: now also R11.1
- net Vout: now also C7.2
- net GPIO22: now reaches IC1.36 (IO22)
- net GPIO23: now reaches IC1.37 (IO23)
