File: schematics/tower.kicad_sch (KiCad schematic)
At the start: 26 parts, among them IC1 ESP32-SOLO-1, J1 216990-0003, J2 Conn_01x06, J3 Conn_01x05, J4 SD_Card, J5 Conn_02x10_Odd_Even, Q1 SS8050-G, Q2 SS8050-G, SW1 SW_Push, SW2 SW_Push

Commit message: think Ive finished the schematics
Parts:
- IC1: footprint Mouser:ESP32SOLO1 -> RF_Module:ESP32-WROOM-32
- J2: footprint Connector_PinSocket_1.00mm:PinSocket_1x06_P1.00mm_Vertical -> Connector_PinSocket_2.54mm:PinSocket_1x06_P2.54mm_Vertical
- R6, R7: footprint Resistor_SMD:R_0201_0603Metric -> Resistor_SMD:R_0805_2012Metric
Changed lines of the file:
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@@
     (property "Reference" "IC1" (id 0) (at 187.96 36.449 0))
     (property "Value" "ESP32-SOLO-1" (id 1) (at 187.96 38.7604 0))
-    (property "Footprint" "Mouser:ESP32SOLO1" (id 2) (at 201.93 40.64 0)
+    (property "Footprint" "RF_Module:ESP32-WROOM-32" (id 2) (at 201.93 40.64 0)
       (effects (font (size 1.27 1.27)) (justify left) hide)
     )
@@
       (effects (font (size 1.27 1.27)) (justify left))
     )
-    (property "Footprint" "Connector_PinSocket_1.00mm:PinSocket_1x06_P1.00mm_Vertical" (id 2) (at 95.25 118.11 0)
+    (property "Footprint" "Connector_PinSocket_2.54mm:PinSocket_1x06_P2.54mm_Vertical" (id 2) (at 95.25 118.11 0)
       (effects (font (size 1.27 1.27)) hide)
     )
@@
       (effects (font (size 1.27 1.27)) (justify left))
     )
-    (property "Footprint" "Resistor_SMD:R_0201_0603Metric" (id 2) (at 137.922 105.41 90)
+    (property "Footprint" "Resistor_SMD:R_0805_2012Metric" (id 2) (at 137.922 105.41 90)
       (effects (font (size 1.27 1.27)) hide)
     )
@@
     (property "Reference" "R7" (id 0) (at 90.3478 66.04 90))
     (property "Value" "0" (id 1) (at 88.0364 66.04 90))
-    (property "Footprint" "Resistor_SMD:R_0201_0603Metric" (id 2) (at 86.868 66.04 90)
+    (property "Footprint" "Resistor_SMD:R_0805_2012Metric" (id 2) (at 86.868 66.04 90)
       (effects (font (size 1.27 1.27)) hide)
     )
@@
   (symbol (lib_id "power:GND") (at 166.37 39.37 180) (unit 1)
     (in_bom yes) (on_board yes)
-    (property "Reference" "#PWR?" (id 0) (at 166.37 33.02 0)
+    (property "Reference" "#PWR0101" (id 0) (at 166.37 33.02 0)
       (effects (font (size 1.27 1.27)) hide)
     )
@@
     )
     (path "/00000000-0000-0000-0000-0000622062dd"
-      (reference "#PWR?") (unit 1) (value "GND") (footprint "")
+      (reference "#PWR0101") (unit 1) (value "GND") (footprint "")
     )
     (path "/00000000-0000-0000-0000-00006220cbe7"
@@
     )
     (path "/00000000-0000-0000-0000-00006209664c"
-      (reference "IC1") (unit 1) (value "ESP32-SOLO-1") (footprint "Mouser:ESP32SOLO1")
+      (reference "IC1") (unit 1) (value "ESP32-SOLO-1") (footprint "RF_Module:ESP32-WROOM-32")
     )
     (path "/00000000-0000-0000-0000-0000622e8087"
@@
     )
     (path "/00000000-0000-0000-0000-0000621305fa"
-      (reference "J2") (unit 1) (value "Conn_01x06") (footprint "Connector_PinSocket_1.00mm:PinSocket_1x06_P1.00mm_Vertical")
+      (reference "J2") (unit 1) (value "Conn_01x06") (footprint "Connector_PinSocket_2.54mm:PinSocket_1x06_P2.54mm_Vertical")
     )
     (path "/00000000-0000-0000-0000-00006226446b"
@@
     )
     (path "/00000000-0000-0000-0000-0000621f10c3"
-      (reference "R6") (unit 1) (value "0") (footprint "Resistor_SMD:R_0201_0603Metric")
+      (reference "R6") (unit 1) (value "0") (footprint "Resistor_SMD:R_0805_2012Metric")
     )
     (path "/00000000-0000-0000-0000-0000621f3c14"
-      (reference "R7") (unit 1) (value "0") (footprint "Resistor_SMD:R_0201_0603Metric")
+      (reference "R7") (unit 1) (value "0") (footprint "Resistor_SMD:R_0805_2012Metric")
     )
     (path "/00000000-0000-0000-0000-00006220c472"

Commit message: final pcbs and schematics
Parts:
- removed J1: 216990-0003, Mouser:2169900003, symbol Mouser:216990-0003
- added J1: USB_B_Micro, Connector_USB:USB_Micro-B_Molex-105017-0001, symbol Connector:USB_B_Micro
- added R8: 10k, Resistor_SMD:R_0805_2012Metric, symbol Device:R
- R1: value 20 -> 10k
Connections:
- net EN: now also R8.1
- net GND: now also J1.5 (GND), J1.6 (Shield)
- net GPIO0: now also R1.1
- net VOUT: now also R1.2, R8.2; no longer J2.3 (Pin_3)
- net at D1.2: now also J1.1 (VBUS); no longer R1.1
- no-connect marks 0 -> 1
Other:
- moved on the sheet: D1
